File: DMH_Dual_VCA_Mk2_PANEL/DMH_Dual_VCA_Mk2_PANEL.kicad_sch (KiCad schematic)
At the start: 19 parts, among them J0 Panel_GND_Solder_Wire_Pad

Commit message: Finished panel
Parts:
- added H19: Mix, SynthStuff:Jack_6.35mm_Cutout_Output_v6, symbol SynthStuff:MountingHole_Jack6.35mm_v2
- H10: value CV 2 -> CV A 2
- H11: value Output -> Out A
- H12: value Offset -> Offset B; footprint SynthStuff:Pot_Cutout_Small -> SynthStuff:Pot_Cutout_Tiny
- H13: value CV 1 Amt -> CV B 1 Amt
- H14: value CV 2 Amt -> CV B 2 Amt
- H15: value Input -> Input B
- H16: value Output -> Out B
- H17: value CV 1 -> CV B 1
- H18: value CV 2 -> CV B 2
- H5: value Offset -> Offset A; footprint SynthStuff:Pot_Cutout_Small -> SynthStuff:Pot_Cutout_Tiny
- H6: value CV 1 Amt -> CV A 1 Amt
- H7: value CV 2 Amt -> CV A 2 Amt
- H8: value Input -> Input A
- H9: value CV 1 -> CV A 1
Connections:
- net GND: now also H19.1
Changed lines of the file:
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@@
+	)
+	(junction
+		(at 50.8 228.6)
+		(diameter 0)
+		(color 0 0 0 0)
 	)
 	(junction
@@
 	(wire
 		(pts
-			(xy 50.8 215.9) (xy 50.8 219.71)
+			(xy 50.8 215.9) (xy 50.8 228.6)
 		)
 		(stroke
@@
 	(wire
 		(pts
+			(xy 50.8 228.6) (xy 59.69 228.6)
+		)
+		(stroke
+			(width 0)
+			(type default)
+		)
+	)
+	(wire
+		(pts
 			(xy 76.2 190.5) (xy 76.2 203.2)
 		)
@@
 		(pts
 			(xy 27.94 259.08) (xy 24.13 259.08)
+		)
+		(stroke
+			(width 0)
+			(type default)
+		)
+	)
+	(wire
+		(pts
+			(xy 50.8 228.6) (xy 50.8 240.03)
 		)
 		(stroke
@@
 			)
 		)
-		(property "Value" "CV 2 Amt"
+		(property "Value" "CV B 2 Amt"
 			(at 104.14 177.7999 0)
 			(effects
@@
 			)
 		)
-		(property "Value" "CV 1"
+		(property "Value" "CV B 1"
 			(at 78.74 215.8999 0)
 			(effects
@@
 			)
 		)
-		(property "Value" "Offset"
+		(property "Value" "Offset A"
 			(at 91.44 88.8999 0)
 			(effects
@@
 			)
 		)
-		(property "Footprint" "SynthStuff:Pot_Cutout_Small"
+		(property "Footprint" "SynthStuff:Pot_Cutout_Tiny"
 			(at 88.9 90.17 0)
 			(effects
@@
 			)
 		)
-		(property "Value" "Input"
+		(property "Value" "Input A"
 			(at 66.04 126.9999 0)
 			(effects
@@
 			)
 		)
-		(property "Value" "CV 1"
+		(property "Value" "CV A 1"
 			(at 78.74 139.6999 0)
 			(effects
@@
 			)
 		)
-		(property "Value" "Input"
+		(property "Value" "Input B"
 			(at 66.04 203.1999 0)
 			(effects
@@
 			)
 		)
-		(property "Value" "CV 2 Amt"
+		(property "Value" "CV A 2 Amt"
 			(at 104.14 101.5999 0)
 			(effects
@@
 	(symbol
 		(lib_id "power:GND")
-		(at 50.8 219.71 0)
+		(at 50.8 240.03 0)
 		(unit 1)
 		(exclude_from_sim no)
@@
 		(fields_autoplaced yes)
 		(property "Reference" "#PWR02"
-			(at 50.8 226.06 0)
+			(at 50.8 246.38 0)
 			(effects
 				(font
@@
 		)
 		(property "Value" "GND"
-			(at 50.8 224.79 0)
+			(at 50.8 245.11 0)
 			(effects
 				(font
@@
 		)
 		(property "Footprint" ""
-			(at 50.8 219.71 0)
+			(at 50.8 240.03 0)
 			(effects
 				(font
@@
 		)
 		(property "Datasheet" ""
-			(at 50.8 219.71 0)
+			(at 50.8 240.03 0)
 			(effects
 				(font
@@
 		)
 		(property "Description" "Power symbol creates a global label with name \"GND\" , ground"
-			(at 50.8 219.71 0)
+			(at 50.8 240.03 0)
 			(effects
 				(font
@@
 			)
 		)
-		(property "Value" "CV 2"
+		(property "Value" "CV B 2"
 			(at 104.14 215.8999 0)
 			(effects
@@
 			)
 		)
-		(property "Value" "CV 2"
+		(property "Value" "CV A 2"
 			(at 104.14 139.6999 0)
 			(effects
@@
 			)
 		)
-		(property "Value" "Output"
+		(property "Value" "Out A"
 			(at 116.84 126.9999 0)
 			(effects
@@
 			)
 		)
-		(property "Value" "CV 1 Amt"
+		(property "Value" "CV A 1 Amt"
 			(at 78.74 101.5999 0)
 			(effects
@@
 			)
 		)
-		(property "Value" "CV 1 Amt"
+		(property "Value" "CV B 1 Amt"
 			(at 78.74 177.7999 0)
 			(effects
@@
 				(path "/a552705f-a9fe-462e-9913-5cfcc08b233c"
 					(reference "H13")
+					(unit 1)
+				)
+			)
+		)
+	)
+	(symbol
+		(lib_id "SynthStuff:MountingHole_Jack6.35mm_v2")
+		(at 63.5 228.6 0)
+		(unit 1)
+		(exclude_from_sim no)
+		(in_bom no)
+		(on_board yes)
+		(dnp no)
+		(fields_autoplaced yes)
+		(property "Reference" "H19"
+			(at 66.04 226.0599 0)
+			(effects
+				(font
+					(size 1.27 1.27)
+				)
+				(justify left)
+			)
+		)
+		(property "Value" "Mix"
+			(at 66.04 228.5999 0)
+			(effects
+				(font
+					(size 1.27 1.27)
+				)
+				(justify left)
+			)
+		)
+		(property "Footprint" "SynthStuff:Jack_6.35mm_Cutout_Output_v6"
+			(at 63.5 228.6 0)
+			(effects
+				(font
+					(size 1.27 1.27)
+				)
+				(hide yes)
+			)
+		)
+		(property "Datasheet" "~"
+			(at 63.5 228.6 0)
+			(effects
+				(font
+					(size 1.27 1.27)
+				)
+				(hide yes)
+			)
+		)
+		(property "Description" "Jack 6.35mm"
+			(at 66.04 231.1399 0)
+			(effects
+				(font
+					(size 1.27 1.27)
+				)
+				(justify left)
+			)
+		)
+		(pin "1"
+		)
+		(instances
+			(project "DMH_Dual_VCA_Mk2_PANEL"
+				(path "/a552705f-a9fe-462e-9913-5cfcc08b233c"
+					(reference "H19")
 					(unit 1)
 				)
@@
 			)
 		)
-		(property "Value" "Offset"
+		(property "Value" "Offset B"
 			(at 91.44 165.0999 0)
 			(effects
@@
 			)
 		)
-		(property "Footprint" "SynthStuff:Pot_Cutout_Small"
+		(property "Footprint" "SynthStuff:Pot_Cutout_Tiny"
 			(at 88.9 166.37 0)
 			(effects
@@
 			)
 		)
-		(property "Value" "Output"
+		(property "Value" "Out B"
 			(at 116.84 203.1999 0)
 			(effects
