File: DMH_Dual_VCA_Mk2_PCB_1/Power.kicad_sch (KiCad schematic)
At the start: 13 parts, among them J100 IDC_02x05, U1 TL074, U2 TL074

Commit message: Finished schematic for PCB 1
Parts:
- added U3: TL072, symbol Amplifier_Operational:TL072
- renumbered C5 to C3, C6 to C4, C7 to C5, C8 to C6, C3 to C7, C4 to C8
Connections:
- net +12V: now also U3.8 (V+)
- net -12V: now also U3.4 (V-)
Other:
- moved on the sheet: C7, C8

Commit message: Routed PCB 1
Parts:
- U2: footprint (none) -> Package_DIP:DIP-14_W7.62mm_Socket
- U3: footprint (none) -> Package_DIP:DIP-8_W7.62mm_Socket
Changed lines of the file:
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@@
+		)
+	)
+	(netclass_flag ""
+		(length 2.54)
+		(shape round)
+		(at 100.33 185.42 180)
+		(fields_autoplaced yes)
+		(effects
+			(font
+				(size 1.27 1.27)
+			)
+			(justify right bottom)
+		)
+		(property "Netclass" "Power"
+			(at 101.0285 187.96 0)
+			(effects
+				(font
+					(size 1.27 1.27)
+				)
+				(justify left)
+			)
+		)
+		(property "Component Class" ""
+			(at -1.27 -2.54 0)
+			(effects
+				(font
+					(size 1.27 1.27)
+					(italic yes)
+				)
+			)
+		)
+	)
+	(netclass_flag ""
+		(length 2.54)
+		(shape round)
+		(at 100.33 175.26 0)
+		(fields_autoplaced yes)
+		(effects
+			(font
+				(size 1.27 1.27)
+			)
+			(justify left bottom)
+		)
+		(property "Netclass" "Power"
+			(at 101.0285 172.72 0)
+			(effects
+				(font
+					(size 1.27 1.27)
+				)
+				(justify left)
+			)
+		)
+		(property "Component Class" ""
+			(at -77.47 21.59 0)
+			(effects
+				(font
+					(size 1.27 1.27)
+					(italic yes)
+				)
+			)
 		)
 	)
@@
 			)
 		)
-		(property "Footprint" ""
+		(property "Footprint" "Package_DIP:DIP-8_W7.62mm_Socket"
 			(at 104.14 120.65 0)
 			(effects
@@
 			)
 		)
-		(property "Footprint" ""
+		(property "Footprint" "Package_DIP:DIP-14_W7.62mm_Socket"
 			(at 77.47 118.11 0)
 			(effects
