File: DMH_Dual_VCA_Mk2_PCB_2/DMH_Dual_VCA_Mk2_PCB_2.kicad_sch (KiCad schematic)
At the start: 0 parts

Commit message: Routed PCB 3
Connections:
- no-connect marks 0 -> 15
Other:
- removed sheet Core Circuit A
- removed sheet Core Circuit B
- removed sheet Mixer
- removed sheet Power
